File: smpsu.sch (KiCad schematic (older format))
At the start: 12 parts, among them J1 Screw_Terminal_01x02, J2 Screw_Terminal_01x02, U1 LM2676SX-ADJ_NOPB

Commit message: WIP: redesign for better stability
Parts:
- removed J1: Screw_Terminal_01x02, 282837-2:TE_282837-2, symbol Connector:Screw_Terminal_01x02
- added J1: PJ-037B, Project:CUI_PJ-037B, symbol PJ-037B:PJ-037B
- RV1: footprint Potentiometer_THT:Potentiometer_Bourns_3296W_Vertical -> Potentiometer_THT:Potentiometer_Vishay_T73XW_Horizontal
Connections:
- net GND: now also J2.1 (Pin_1), J1.2; no longer J2.2 (Pin_2)
- net at C1.1, C2.1, U1.2 (Input): now also J1.1
- net at C4.1, L1.2, RV1.2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: now also J2.2 (Pin_2); no longer J2.1 (Pin_1)
Changed lines of the file:
@@
 F 0 "RV1" V 7186 2400 50  0000 C CNN
 F 1 "30k" V 7095 2400 50  0000 C CNN
-F 2 "Potentiometer_THT:Potentiometer_Bourns_3296W_Vertical" H 7300 2400 50  0001 C CNN
+F 2 "Potentiometer_THT:Potentiometer_Vishay_T73XW_Horizontal" H 7300 2400 50  0001 C CNN
 F 3 "~" H 7300 2400 50  0001 C CNN
 	1    7300 2400
@@
 Connection ~ 6550 3100
 $Comp
-L Connector:Screw_Terminal_01x02 J1
-U 1 1 5BF8EB16
-P 3550 3000
-F 0 "J1" H 3550 2800 50  0000 C CNN
-F 1 "Screw_Terminal_01x02" H 3470 2766 50  0001 C CNN
-F 2 "282837-2:TE_282837-2" H 3550 3000 50  0001 C CNN
-F 3 "~" H 3550 3000 50  0001 C CNN
-	1    3550 3000
-	-1   0    0    1
-$EndComp
-$Comp
 L Connector:Screw_Terminal_01x02 J2
 U 1 1 5BF8EB9A
-P 8450 2900
-F 0 "J2" H 8400 3000 50  0000 L CNN
-F 1 "Screw_Terminal_01x02" H 8530 2801 50  0001 L CNN
-F 2 "282837-2:TE_282837-2" H 8450 2900 50  0001 C CNN
-F 3 "~" H 8450 2900 50  0001 C CNN
-	1    8450 2900
-	1    0    0    -1
+P 8450 3000
+F 0 "J2" H 8400 3100 50  0000 L CNN
+F 1 "Screw_Terminal_01x02" H 8530 2901 50  0001 L CNN
+F 2 "282837-2:TE_282837-2" H 8450 3000 50  0001 C CNN
+F 3 "~" H 8450 3000 50  0001 C CNN
+	1    8450 3000
+	1    0    0    1
 $EndComp
 Wire Wire Line
-	3750 2900 4150 2900
+	3650 2900 4150 2900
 Connection ~ 4150 2900
 Wire Wire Line
-	3750 3000 3750 3750
-Wire Wire Line
-	3750 3750 4150 3750
+	3650 3750 4150 3750
 Connection ~ 4150 3750
 Wire Wire Line
@@
 	8250 3750 7550 3750
 Connection ~ 7550 3750
+$Comp
+L PJ-037B:PJ-037B J1
+U 1 1 5C1A6E01
+P 3450 3000
+F 0 "J1" H 3419 3340 50  0000 C CNN
+F 1 "PJ-037B" H 3419 3249 50  0000 C CNN
+F 2 "Project:CUI_PJ-037B" H 3450 3000 50  0001 L BNN
+F 3 "Manufacturer recommendations" H 3450 3000 50  0001 L BNN
+F 4 "CUI INC" H 3450 3000 50  0001 L BNN "Field4"
+	1    3450 3000
+	1    0    0    -1
+$EndComp
+Wire Wire Line
+	3650 3100 3650 3750
 $EndSCHEMATC
